File: ferris.sch (KiCad schematic (older format))
At the start: 69 parts, among them K0_0 KEYSW, K0_1 KEYSW, K0_2 KEYSW, K0_3 KEYSW, K0_4 KEYSW, K0_5 KEYSW, K0_6 KEYSW, K0_7 KEYSW, K0_8 KEYSW, K0_9 KEYSW, K1_0 KEYSW, K1_1 KEYSW, K1_2 KEYSW, K1_3 KEYSW, K1_4 KEYSW, K1_5 KEYSW, K1_6 KEYSW, K1_7 KEYSW, K1_8 KEYSW, K1_9 KEYSW, K2_0 KEYSW, K2_1 KEYSW, K2_2 KEYSW, K2_3 KEYSW, K2_4 KEYSW, K2_5 KEYSW, K2_6 KEYSW, K2_7 KEYSW, K2_8 KEYSW, K2_9 KEYSW, K3_3 KEYSW, K3_4 KEYSW, K3_5 KEYSW, K3_6 KEYSW, U1 ProMicro_r

Commit message: Symmetry
Parts:
- D0_0, D0_1, D0_2, D0_3, D0_4, D0_5, D0_6, D0_7, D0_8, D0_9, D1_0, D1_1, D1_2, D1_3, D1_4, D1_5, D1_6, D1_7, D1_8, D1_9, D2_0, D2_1, D2_2, D2_3, D2_4, D2_5, D2_6, D2_7, D2_8, D2_9, D3_3, D3_4, D3_5, D3_6: symbol Device:D -> ferris-rescue:D-Device
- K0_0, K0_1, K0_2, K0_3, K0_4, K0_5, K0_6, K0_7, K0_8, K0_9, K1_0, K1_1, K1_2, K1_3, K1_4, K1_5, K1_6, K1_7, K1_8, K1_9, K2_0, K2_1, K2_2, K2_3, K2_4, K2_5, K2_6, K2_7, K2_8, K2_9, K3_3, K3_4, K3_5, K3_6: symbol kbd:SW_PUSH -> ferris-rescue:SW_PUSH-kbd
- U1: symbol kbd:ProMicro_r -> ferris-rescue:ProMicro_r-kbd
